File: keyboard_design_example.kicad_pcb (KiCad board)
At the start: 2 copper layers, 24 parts, among them SW1 SW_PUSH, U1 ATmega32U4-AU, Y1 16MHz

Commit message: Update
Parts:
- moved R2 149.3 mm to (38.9, 57.9), turned to 270 degrees
- moved USB1 143.9 mm to (37.0, 49.2), turned to 270 degrees
- moved C6 132.8 mm to (53.2, 50.8), turned to 90 degrees
- moved R4 130.2 mm to (45.4, 54.5), turned to 270 degrees
- moved C4 116.6 mm to (53.2, 73.7)
- moved R3 107.3 mm to (67.5, 68.9), turned to 270 degrees
- moved C3 21.0 mm to (60.8, 73.7)
- moved C2 16.6 mm to (66.9, 54.6), turned to 270 degrees
- moved SW1 15.7 mm to (36.5, 79.4)
- moved C7 11.4 mm to (45.6, 66.0), turned to 0 degrees
- moved D1 11.1 mm to (86.5, 57.1), turned to 270 degrees
- moved D2 11.1 mm to (105.6, 57.1), turned to 270 degrees
- moved C1 10.2 mm to (48.9, 54.5)
- moved F1 9.24 mm to (29.4, 62.7)
- moved C5 8.59 mm to (60.8, 50.8)
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Other:
- net class Default: clearance 0.2 -> 7.874016; trace_width 0.25 -> 0.254; via_dia 0.8 -> 31.49606; via_drill 0.4 -> 15.74803
- net class Power added: clearance 7.874016, trace_width 0.381, via_dia 31.49606, via_drill 15.74803
- rule trace_clearance: 0.2 -> 7.874016

Commit message: Update and work
Parts:
- moved R1 4.76 mm to (38.9, 57.9), turned to 90 degrees
- moved R2 3.17 mm to (35.7, 57.9), turned to 90 degrees
- moved C7 1.75 mm to (45.6, 64.3)
Connections:
- C1 pad 2: +5V -> GND
- C2 pad 2: +5V -> GND
- C3 pad 2: +5V -> GND
- C4 pad 2: +5V -> GND
- C5 pad 2: +5V -> GND
- C6 pad 2: +5V -> GND
- C7 pad 2: +5V -> GND
- R4 pad 1: +5V -> GND
- SW1 pad 1: +5V -> GND
- U1 pad 15: +5V -> GND
- U1 pad 23: +5V -> GND
- U1 pad 35: +5V -> GND
- U1 pad 43: +5V -> GND
- U1 pad 5: +5V -> GND
- USB1 pad 1: +5V -> GND
- Y1 pad 2: +5V -> GND
- Y1 pad 4: +5V -> GND
Routing:
- net Net-(R2-Pad1): track 0.00 -> 16.8 mm
- net Net-(R1-Pad1): track 0.00 -> 14.3 mm
- net D+: track 0.00 -> 3.84 mm
- net D-: track 0.00 -> 3.78 mm
- net GND: track 0.00 -> 2.71 mm
Other:
- net class Default: clearance 7.874016 -> 0.25
- net class Power: clearance 7.874016 -> 0.3
- rule trace_clearance: 7.874016 -> 0.25

Commit message: Update
Working on pcb organization
Parts:
- added D5: SOD-123, Diode_SMD:D_SOD-123, F.Cu at (145.3, 109.5)
- added D6: SOD-123, Diode_SMD:D_SOD-123, F.Cu at (164.3, 109.5)
- added D7: SOD-123, Diode_SMD:D_SOD-123, F.Cu at (126.2, 128.6)
- added D8: SOD-123, Diode_SMD:D_SOD-123, F.Cu at (145.3, 128.6)
- added D9: SOD-123, Diode_SMD:D_SOD-123, F.Cu at (164.3, 128.6)
- added MX5: MX-NoLED, MX_Only:MXOnly-1U-NoLED, F.Cu at (137.3, 109.5)
- added MX6: MX-NoLED, MX_Only:MXOnly-1U-NoLED, F.Cu at (156.4, 109.5)
- added MX7: MX-NoLED, MX_Only:MXOnly-1U-NoLED, F.Cu at (118.3, 128.6)
- added MX8: MX-NoLED, MX_Only:MXOnly-1U-NoLED, F.Cu at (137.3, 128.6)
- added MX9: MX-NoLED, MX_Only:MXOnly-1U-NoLED, F.Cu at (156.4, 128.6)
- moved SW1 79.7 mm to (94.5, 134.1)
- moved D3 79.1 mm to (164.3, 90.5)
- moved MX3 79.1 mm to (156.4, 90.5)
- moved C7 73.9 mm to (112.6, 33.2)
- moved R2 73.5 mm to (106.9, 39.5), turned to 0 degrees
- moved Y1 66.8 mm to (72.2, 115.9)
- moved C3 59.2 mm to (106.9, 36.5)
- moved F1 56.4 mm to (73.0, 98.4)
- moved C1 56.4 mm to (64.3, 108.7)
- moved R1 52.9 mm to (91.3, 51.0), turned to 0 degrees
- moved D1 51.8 mm to (126.2, 90.5)
- moved D2 51.8 mm to (145.3, 90.5)
- moved MX1 51.8 mm to (118.3, 90.5)
- moved MX2 51.8 mm to (137.3, 90.5)
- moved C6 49.3 mm to (102.0, 43.5), turned to 0 degrees
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Connections:
- D2 pad 1: ROW1 -> ROW0
- MX2 pad 1: COL0 -> COL1
- MX3 pad 1: COL1 -> COL2
- MX4 pad 1: COL1 -> COL0
- U1 pad 27: ROW0 -> Net-(U1-Pad27)
- U1 pad 28: COL1 -> Net-(U1-Pad28)
- U1 pad 29: COL0 -> Net-(U1-Pad29)
- U1 pad 30: ROW1 -> Net-(U1-Pad30)
Routing:
- net Net-(R2-Pad1): track 16.8 -> 0.00 mm
- net Net-(R1-Pad1): track 14.3 -> 0.00 mm
- net D+: track 3.84 -> 0.00 mm
- net D-: track 3.78 -> 0.00 mm
- net GND: track 2.71 -> 0.00 mm

Commit message: Update
stuff
Parts:
- moved C7 119.1 mm to (50.8, 134.9)
- moved C6 100.7 mm to (50.8, 130.2)
- moved C3 97.2 mm to (50.8, 115.9)
- moved C5 80.3 mm to (50.8, 125.4)
- moved C2 79.2 mm to (50.8, 111.1)
- moved R2 74.6 mm to (51.6, 89.7)
- moved C4 73.4 mm to (51.0, 120.7)
- moved R3 57.2 mm to (51.6, 94.5)
- moved R4 52.5 mm to (51.5, 99.2)
- moved R1 52.2 mm to (51.6, 84.9)
- moved SW1 47.0 mm to (50.8, 151.6)
- moved Y1 34.6 mm to (51.6, 143.7)
- moved F1 28.7 mm to (51.6, 79.4), turned to 180 degrees
- moved USB1 25.6 mm to (51.6, 69.1)
- moved C1 13.5 mm to (51.0, 106.4), turned to 0 degrees
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Changed lines of the file:
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@@
   )
   (module Crystal:Crystal_SMD_3225-4Pin_3.2x2.5mm (layer F.Cu)
-    (at 72.23125 115.8875)
+    (at 51.59375 143.66875)
     (descr "SMD Crystal SERIES SMD3225/4 http://www.txccrystal.com/images/pdf/7m-accuracy.pdf, 3.2x2.5mm^2 package")
     (tags "SMD SMT crystal")
@@
   )
   (module random-keyboard-parts:Molex-0548190589 (layer F.Cu)
-    (at 73.81875 81.75625 270)
+    (at 51.59375 69.05625 270)
     (attr smd)
     (fp_text reference USB1 (at 2.032 0) (layer F.SilkS)
@@
   )
   (module Package_QFP:TQFP-44_10x10mm_P0.8mm (layer F.Cu)
-    (at 88.10625 101.6)
+    (at 84.1375 109.5375)
     (descr "44-Lead Plastic Thin Quad Flatpack (PT) - 10x10x1.0 mm Body [TQFP] (see Microchip Packaging Specification 00000049BS.pdf)")
     (tags "QFP 0.8")
@@
   )
   (module random-keyboard-parts:SKQG-1155865 (layer F.Cu)
-    (at 94.45625 134.14375)
+    (at 50.8 151.60625)
     (attr smd)
     (fp_text reference SW1 (at 0 4.064) (layer F.SilkS)
@@
   )
   (module Resistor_SMD:R_0805_2012Metric (layer F.Cu)
-    (at 86.98625 60.6075)
+    (at 51.475 99.21875)
     (descr "Resistor SMD 0805 (2012 Metric), square (rectangular) end terminal, IPC_7351 nominal, (Body size source: IPC-SM-782 page 72, https://www.pcb-3d.com/wordpress/wp-content/uploads/ipc-sm-782a_amendment_1_and_2.pdf), generated with kicad-footprint-generator")
     (tags resistor)
@@
   )
   (module Resistor_SMD:R_0805_2012Metric (layer F.Cu)
-    (at 91.93625 53.9175)
+    (at 51.59375 94.45625)
     (descr "Resistor SMD 0805 (2012 Metric), square (rectangular) end terminal, IPC_7351 nominal, (Body size source: IPC-SM-782 page 72, https://www.pcb-3d.com/wordpress/wp-content/uploads/ipc-sm-782a_amendment_1_and_2.pdf), generated with kicad-footprint-generator")
     (tags resistor)
@@
   )
   (module Resistor_SMD:R_0805_2012Metric (layer F.Cu)
-    (at 106.85625 39.5275)
+    (at 51.59375 89.69375)
     (descr "Resistor SMD 0805 (2012 Metric), square (rectangular) end terminal, IPC_7351 nominal, (Body size source: IPC-SM-782 page 72, https://www.pcb-3d.com/wordpress/wp-content/uploads/ipc-sm-782a_amendment_1_and_2.pdf), generated with kicad-footprint-generator")
     (tags resistor)
@@
   )
   (module Resistor_SMD:R_0805_2012Metric (layer F.Cu)
-    (at 91.28625 50.9675)
+    (at 51.59375 84.93125)
     (descr "Resistor SMD 0805 (2012 Metric), square (rectangular) end terminal, IPC_7351 nominal, (Body size source: IPC-SM-782 page 72, https://www.pcb-3d.com/wordpress/wp-content/uploads/ipc-sm-782a_amendment_1_and_2.pdf), generated with kicad-footprint-generator")
     (tags resistor)
@@
   )
   (module Fuse:Fuse_1206_3216Metric (layer F.Cu)
-    (at 73.025 98.425 90)
+    (at 51.59375 79.375 180)
     (descr "Fuse SMD 1206 (3216 Metric), square (rectangular) end terminal, IPC_7351 nominal, (Body size source: http://www.tortai-tech.com/upload/download/2011102023233369053.pdf), generated with kicad-footprint-generator")
     (tags fuse)
     (attr smd)
-    (fp_text reference F1 (at 0 -1.82 90) (layer F.SilkS)
-      (effects (font (size 1 1) (thickness 0.15)))
-    )
-    (fp_text value Polyfuse_Small (at 0 1.82 90) (layer F.Fab)
-      (effects (font (size 1 1) (thickness 0.15)))
-    )
-    (fp_text user %R (at 0 0 90) (layer F.Fab)
+    (fp_text reference F1 (at 0 -1.82) (layer F.SilkS)
+      (effects (font (size 1 1) (thickness 0.15)))
+    )
+    (fp_text value Polyfuse_Small (at 0 1.82) (layer F.Fab)
+      (effects (font (size 1 1) (thickness 0.15)))
+    )
+    (fp_text user %R (at 0 0) (layer F.Fab)
       (effects (font (size 0.8 0.8) (thickness 0.12)))
     )
@@
     (fp_line (start 2.28 -1.12) (end 2.28 1.12) (layer F.CrtYd) (width 0.05))
     (fp_line (start 2.28 1.12) (end -2.28 1.12) (layer F.CrtYd) (width 0.05))
-    (pad 2 smd roundrect (at 1.4 0 90) (size 1.25 1.75) (layers F.Cu F.Paste F.Mask) (roundrect_rratio 0.2)
+    (pad 2 smd roundrect (at 1.4 0 180) (size 1.25 1.75) (layers F.Cu F.Paste F.Mask) (roundrect_rratio 0.2)
       (net 11 VCC))
-    (pad 1 smd roundrect (at -1.4 0 90) (size 1.25 1.75) (layers F.Cu F.Paste F.Mask) (roundrect_rratio 0.2)
+    (pad 1 smd roundrect (at -1.4 0 180) (size 1.25 1.75) (layers F.Cu F.Paste F.Mask) (roundrect_rratio 0.2)
       (net 1 +5V))
     (model ${KISYS3DMOD}/Fuse.3dshapes/Fuse_1206_3216Metric.wrl
@@
   )
   (module Capacitor_SMD:C_0805_2012Metric (layer F.Cu)
-    (at 112.62625 33.1975)
+    (at 50.8 134.9375)
     (descr "Capacitor SMD 0805 (2012 Metric), square (rectangular) end terminal, IPC_7351 nominal, (Body size source: IPC-SM-782 page 76, https://www.pcb-3d.com/wordpress/wp-content/uploads/ipc-sm-782a_amendment_1_and_2.pdf, https://docs.google.com/spreadsheets/d/1BsfQQcO9C6DZCsRaXUlFlo91Tg2WpOkGARC1WS5S8t0/edit?usp=sharing), generated with kicad-footprint-generator")
     (tags capacitor)
@@
   )
   (module Capacitor_SMD:C_0805_2012Metric (layer F.Cu)
-    (at 101.95625 43.4875)
+    (at 50.8 130.175)
     (descr "Capacitor SMD 0805 (2012 Metric), square (rectangular) end terminal, IPC_7351 nominal, (Body size source: IPC-SM-782 page 76, https://www.pcb-3d.com/wordpress/wp-content/uploads/ipc-sm-782a_amendment_1_and_2.pdf, https://docs.google.com/spreadsheets/d/1BsfQQcO9C6DZCsRaXUlFlo91Tg2WpOkGARC1WS5S8t0/edit?usp=sharing), generated with kicad-footprint-generator")
     (tags capacitor)
@@
   )
   (module Capacitor_SMD:C_0805_2012Metric (layer F.Cu)
-    (at 87.50625 53.9975)
+    (at 50.8 125.4125)
     (descr "Capacitor SMD 0805 (2012 Metric), square (rectangular) end terminal, IPC_7351 nominal, (Body size source: IPC-SM-782 page 76, https://www.pcb-3d.com/wordpress/wp-content/uploads/ipc-sm-782a_amendment_1_and_2.pdf, https://docs.google.com/spreadsheets/d/1BsfQQcO9C6DZCsRaXUlFlo91Tg2WpOkGARC1WS5S8t0/edit?usp=sharing), generated with kicad-footprint-generator")
     (tags capacitor)
@@
   )
   (module Capacitor_SMD:C_0805_2012Metric (layer F.Cu)
-    (at 87.50625 57.0075)
+    (at 50.95625 120.65)
     (descr "Capacitor SMD 0805 (2012 Metric), square (rectangular) end terminal, IPC_7351 nominal, (Body size source: IPC-SM-782 page 76, https://www.pcb-3d.com/wordpress/wp-content/uploads/ipc-sm-782a_amendment_1_and_2.pdf, https://docs.google.com/spreadsheets/d/1BsfQQcO9C6DZCsRaXUlFlo91Tg2WpOkGARC1WS5S8t0/edit?usp=sharing), generated with kicad-footprint-generator")
     (tags capacitor)
@@
   )
   (module Capacitor_SMD:C_0805_2012Metric (layer F.Cu)
-    (at 106.87625 36.5475)
+    (at 50.8 115.8875)
     (descr "Capacitor SMD 0805 (2012 Metric), square (rectangular) end terminal, IPC_7351 nominal, (Body size source: IPC-SM-782 page 76, https://www.pcb-3d.com/wordpress/wp-content/uploads/ipc-sm-782a_amendment_1_and_2.pdf, https://docs.google.com/spreadsheets/d/1BsfQQcO9C6DZCsRaXUlFlo91Tg2WpOkGARC1WS5S8t0/edit?usp=sharing), generated with kicad-footprint-generator")
     (tags capacitor)
@@
   )
   (module Capacitor_SMD:C_0805_2012Metric (layer F.Cu)
-    (at 97.05625 46.8375)
+    (at 50.8 111.125)
     (descr "Capacitor SMD 0805 (2012 Metric), square (rectangular) end terminal, IPC_7351 nominal, (Body size source: IPC-SM-782 page 76, https://www.pcb-3d.com/wordpress/wp-content/uploads/ipc-sm-782a_amendment_1_and_2.pdf, https://docs.google.com/spreadsheets/d/1BsfQQcO9C6DZCsRaXUlFlo91Tg2WpOkGARC1WS5S8t0/edit?usp=sharing), generated with kicad-footprint-generator")
     (tags capacitor)
@@
   )
   (module Capacitor_SMD:C_0805_2012Metric (layer F.Cu)
-    (at 64.29375 108.74375 270)
+    (at 50.95625 106.3625)
     (descr "Capacitor SMD 0805 (2012 Metric), square (rectangular) end terminal, IPC_7351 nominal, (Body size source: IPC-SM-782 page 76, https://www.pcb-3d.com/wordpress/wp-content/uploads/ipc-sm-782a_amendment_1_and_2.pdf, https://docs.google.com/spreadsheets/d/1BsfQQcO9C6DZCsRaXUlFlo91Tg2WpOkGARC1WS5S8t0/edit?usp=sharing), generated with kicad-footprint-generator")
     (tags capacitor)
     (attr smd)
-    (fp_text reference C1 (at 0 -1.68 90) (layer F.SilkS)
-      (effects (font (size 1 1) (thickness 0.15)))
-    )
-    (fp_text value 0.1uF (at 0 1.68 90) (layer F.Fab)
-      (effects (font (size 1 1) (thickness 0.15)))
-    )
-    (fp_text user %R (at 0 0 90) (layer F.Fab)
+    (fp_text reference C1 (at 0 -1.68) (layer F.SilkS)
+      (effects (font (size 1 1) (thickness 0.15)))
+    )
+    (fp_text value 0.1uF (at 0 1.68) (layer F.Fab)
+      (effects (font (size 1 1) (thickness 0.15)))
+    )
+    (fp_text user %R (at 0 0) (layer F.Fab)
       (effects (font (size 0.5 0.5) (thickness 0.08)))
     )
@@
     (fp_line (start 1.7 -0.98) (end 1.7 0.98) (layer F.CrtYd) (width 0.05))
     (fp_line (start 1.7 0.98) (end -1.7 0.98) (layer F.CrtYd) (width 0.05))
-    (pad 2 smd roundrect (at 0.95 0 270) (size 1 1.45) (layers F.Cu F.Paste F.Mask) (roundrect_rratio 0.25)
-      (net 44 GND))
-    (pad 1 smd roundrect (at -0.95 0 270) (size 1 1.45) (layers F.Cu F.Paste F.Mask) (roundrect_rratio 0.25)
+    (pad 2 smd roundrect (at 0.95 0) (size 1 1.45) (layers F.Cu F.Paste F.Mask) (roundrect_rratio 0.25)
+      (net 44 GND))
+    (pad 1 smd roundrect (at -0.95 0) (size 1 1.45) (layers F.Cu F.Paste F.Mask) (roundrect_rratio 0.25)
       (net 1 +5V))
     (model ${KISYS3DMOD}/Capacitor_SMD.3dshapes/C_0805_2012Metric.wrl

Commit message: Update
Did the crystal tracing POGGERS
Parts:
- C1, C2, C3, C4, C5, C6, C7, F1, R1, R2, R3, R4, SW1, U1, USB1, Y1: moved to B.Cu
- moved F1 76.6 mm to (43.7, 155.6), turned to 270 degrees
- moved Y1 62.3 mm to (95.2, 99.2)
- moved C6 58.1 mm to (100.0, 99.2), turned to 90 degrees
- moved R3 48.6 mm to (47.6, 142.9)
- moved C5 47.6 mm to (90.5, 99.2), turned to 270 degrees
- moved R4 39.1 mm to (47.5, 138.1)
- moved C7 32.8 mm to (46.8, 102.4)
- moved C1 24.9 mm to (46.8, 131.0)
- moved SW1 24.9 mm to (57.9, 127.8), turned to 180 degrees
- moved USB1 22.7 mm to (69.8, 82.5)
- moved R2 19.2 mm to (70.6, 92.1), turned to 90 degrees
- moved R1 18.1 mm to (68.3, 92.1), turned to 90 degrees
- moved C2 15.6 mm to (46.8, 126.2)
- moved U1 12.1 mm to (96.0, 111.9)
- moved C3 6.83 mm to (46.8, 121.4)
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Routing:
- net ROW2: track 0.00 -> 39.3 mm
- net ROW1: track 0.00 -> 39.3 mm
- net ROW0: track 0.00 -> 39.3 mm
- net COL2: track 0.00 -> 38.1 mm
- net COL1: track 0.00 -> 38.1 mm
- net COL0: track 0.00 -> 38.1 mm
- net GND: track 0.00 -> 27.1 mm
- net Net-(C6-Pad1): track 0.00 -> 13.5 mm
- net Net-(C5-Pad1): track 0.00 -> 9.98 mm
- net Net-(D6-Pad2): track 0.00 -> 6.87 mm
- net Net-(D1-Pad2): track 0.00 -> 6.87 mm
- net Net-(D9-Pad2): track 0.00 -> 6.82 mm
- net Net-(D8-Pad2): track 0.00 -> 6.82 mm
- net Net-(D5-Pad2): track 0.00 -> 6.82 mm
- net Net-(D3-Pad2): track 0.00 -> 6.82 mm
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Other:
- net class Power: trace_width 0.381 -> 0.35

Commit message: Update
Did Stuff
Parts:
- moved R3 67.5 mm to (88.1, 88.9), turned to 270 degrees
- moved R4 65.9 mm to (91.3, 88.9), turned to 270 degrees
- moved F1 49.4 mm to (73.0, 115.9), turned to 180 degrees
- moved SW1 41.4 mm to (99.2, 131.0), turned to 270 degrees
- moved USB1 31.4 mm to (58.7, 111.9), turned to 0 degrees
- moved R1 21.4 mm to (68.3, 113.5), turned to 180 degrees
- moved R2 19.2 mm to (68.3, 111.1), turned to 180 degrees
- moved U1 15.1 mm to (100.8, 97.6)
- moved C5 15.1 mm to (95.2, 84.9)
- moved C6 15.1 mm to (104.8, 84.9)
- moved Y1 15.1 mm to (100.0, 84.9)
- moved C7 9.53 mm to (46.8, 111.9)
Routing:
- net VCC: track 0.00 -> 9.64 mm
- net Net-(R3-Pad2): track 0.00 -> 5.90 mm, vias 0 -> 2

Commit message: Finished
WOOOO I think i finished. Might have to do some updates for fixes but its going good.
Parts:
- D1, D2, D3, D4, D5, D6, D7, D8, D9: moved to B.Cu
- moved C2 60.5 mm to (107.2, 122.2), turned to 90 degrees
- moved C1 55.7 mm to (102.4, 134.9), turned to 180 degrees
- moved R4 45.7 mm to (107.2, 131.8), turned to 90 degrees
- moved C4 43.5 mm to (88.1, 131.0), turned to 270 degrees
- moved C3 43.0 mm to (89.7, 117.5), turned to 90 degrees
- moved C7 42.7 mm to (88.1, 123.0), turned to 180 degrees
- moved R3 28.8 mm to (84.9, 117.5)
- moved U1 28.7 mm to (98.4, 126.2)
- moved C5 28.7 mm to (92.9, 113.5)
- moved C6 28.7 mm to (102.4, 113.5)
- moved Y1 28.7 mm to (97.6, 113.5)
- moved SW1 27.0 mm to (99.2, 104.0)
- moved R2 22.9 mm to (87.3, 98.4)
- moved USB1 22.9 mm to (77.8, 99.2)
- moved R1 22.9 mm to (87.3, 100.8)
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Connections:
- U1 pad 27: Net-(U1-Pad27) -> COL0
- U1 pad 28: Net-(U1-Pad28) -> COL1
- U1 pad 29: Net-(U1-Pad29) -> ROW0
- U1 pad 30: Net-(U1-Pad30) -> COL2
- U1 pad 31: Net-(U1-Pad31) -> ROW1
- U1 pad 32: Net-(U1-Pad32) -> ROW2
Routing:
- net +5V: track 0.00 -> 113.6 mm, vias 0 -> 5
- net COL1: track 38.1 -> 121.7 mm
- net GND: track 27.1 -> 107.0 mm
- net COL2: track 38.1 -> 112.3 mm
- net ROW2: track 39.3 -> 113.1 mm
- net ROW1: track 39.3 -> 109.3 mm
- net ROW0: track 39.3 -> 100.1 mm
- net COL0: track 38.1 -> 96.3 mm
- net Net-(R3-Pad2): track 5.90 -> 49.9 mm
- net Net-(R2-Pad1): track 0.00 -> 40.4 mm
- net Net-(R1-Pad1): track 0.00 -> 38.7 mm
- net Net-(C7-Pad1): track 0.00 -> 6.74 mm
- net Net-(C6-Pad1): track 13.5 -> 9.98 mm
- net Net-(C5-Pad1): track 9.98 -> 13.5 mm
- net VCC: track 9.64 -> 7.87 mm
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Other:
- net class Default: via_dia 31.49606 -> 1; via_drill 15.74803 -> 0.5
- net class Power: via_dia 31.49606 -> 1; via_drill 15.74803 -> 0.5
