File: keyboard_design_example.kicad_pcb (KiCad board)
At the start: 2 copper layers, 34 parts, among them SW1 SW_PUSH, U1 ATmega32U4-AU, Y1 16MHz

Commit message: Update
Still messing with it
Parts:
- SW1: moved to F.Cu
- moved SW1 33.0 mm to (19.8, 111.1)
Routing:
- net GND: track 117.1 -> 144.4 mm, vias 0 -> 1
- net Net-(R3-Pad2): track 49.9 -> 25.0 mm, vias 2 -> 1
- net Net-(C6-Pad1): track 9.98 -> 19.6 mm
- added copper zone on B.Cu, net GND
Other:
- board outline added: 57.1 x 89.7 mm

Commit message: Finished!!!
I finally finished the pcb. It looks great and has my logo on it. Im gonna start my alice board project and try to get this one manufactured.
Parts:
- moved C5 9.52 mm to (37.3, 133.3), turned to 0 degrees
- moved C6 9.52 mm to (37.3, 123.8), turned to 180 degrees
- turned Y1 to 90 degrees
Routing:
- net Net-(C6-Pad1): track 19.6 -> 13.5 mm
- net Net-(C5-Pad1): track 13.8 -> 11.5 mm
- net GND: track 144.4 -> 146.2 mm
Other:
- board text added: "Designed by AltaFour in Colorado"
- board text added: "My wallet hurts less now"
